Commit message: feat(robot_description): 添加机械臂各连杆的碰撞检测配置

File: ros2_ws/src/robot_description/urdf/arm.xacro (robot description, xacro)
@@ -9,4 +9,10 @@
         <material name="grey" />
       </visual>
+      <collision>
+        <geometry>
+          <box size="0.4 0.4 0.1"/>
+        </geometry>
+        <origin xyz="0.0 0.0 0.05" rpy="0.0 0.0 0.0"/>
+      </collision>
     </link>
     <link name="shoulder_link">
@@ -18,4 +24,11 @@
         <material name="blue" />
       </visual>
+      <collision>
+        <geometry>
+          <!-- 用包围盒近似 cylinder: size = (2*radius, 2*radius, length) -->
+          <box size="0.2 0.2 0.5"/>
+        </geometry>
+        <origin xyz="0.0 0.0 0.25" rpy="0.0 0.0 0.0"/>
+      </collision>
     </link>
     <link name="arm_link">
@@ -27,4 +40,11 @@
         <material name="grey" />
       </visual>
+      <collision>
+        <geometry>
+          <!-- cylinder -> box: size = (2*radius, 2*radius, length) -->
+          <box size="0.1 0.1 0.6"/>
+        </geometry>
+        <origin xyz="0.0 0.0 0.3" rpy="0.0 0.0 0.0"/>
+      </collision>
     </link>
     <link name="elbow_link">
@@ -36,4 +56,11 @@
         <material name="blue" />
       </visual>
+      <collision>
+        <geometry>
+          <!-- cylinder -> box -->
+          <box size="0.1 0.1 0.1"/>
+        </geometry>
+        <origin xyz="0.0 0.0 0.05" rpy="0.0 0.0 0.0"/>
+      </collision>
     </link>
     <link name="forearm_link">
@@ -45,4 +72,11 @@
         <material name="grey" />
       </visual>
+      <collision>
+        <geometry>
+          <!-- cylinder -> box -->
+          <box size="0.1 0.1 0.5"/>
+        </geometry>
+        <origin xyz="0.0 0.0 0.25" rpy="0.0 0.0 0.0"/>
+      </collision>
     </link>
 	<link name="wrist_link">
@@ -54,4 +88,10 @@
         <material name="blue" />
       </visual>
+      <collision>
+        <geometry>
+          <box size="0.1 0.1 0.05"/>
+        </geometry>
+        <origin xyz="0.0 0.0 0.025" rpy="0.0 0.0 0.0"/>
+      </collision>
     </link>
 	<link name="hand_link">
@@ -63,6 +103,12 @@
         <material name="grey" />
       </visual>
+      <collision>
+        <geometry>
+          <box size="0.1 0.1 0.02"/>
+        </geometry>
+        <origin xyz="0.0 0.0 0.025" rpy="0.0 0.0 0.0"/>
+      </collision>
     </link>
-	<link name="tool_link" />
+	<link name="tool_link"/>
     <joint name="joint1" type="revolute">
         <parent link="base_link"/>
